File: 2A/Electronique/Schema Electronique 2223/puissance_ok/puissanceok/puissanceok.kicad_sch (KiCad schematic)
At the start: 24 parts, among them J101 Bat 2, J102 Bat 1, J103 AU, J104 Switch, J105 Conn_01x03, J107 Conn_01x02, J108 Conn_01x02, J109 Conn_01x02, J110 Conn_01x02, J111 Conn_01x02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

Commit message: pcb puissance update
Parts:
- removed J105: Conn_01x03, symbol Connector_Generic:Conn_01x03
- removed J107, J108, J109, J110, J111: Conn_01x02, symbol Connector_Generic:Conn_01x02
- removed J112: Conn_01x04, symbol Connector_Generic:Conn_01x04
Other:
- added sheet CONNECTEURS (Connecteurs.kicad_sch)
- note removed: "Connecteur 5.1V"
- note removed: "Connecteur 7.4V - XL320"
- note removed: "Connecteurs"
- note removed: "Lidar"
- note removed: "Phidget Power Supply Stepper"
- moved on the sheet: J113
